File: flex-strip-tester-v7.kicad_pcb (KiCad board)
At the start: 2 copper layers, 67.2 x 11.1 mm, 6 parts, among them J1 Conn_01x01_Female, J2 Conn_01x01_Female

Commit message: try cutout design
Routing:
- net GND: track 41.7 -> 40.0 mm
- net +3V3: track 32.6 -> 31.4 mm
Other:
- outline, holes or cut-outs redrawn
- board text added: "drew@ oshpark.com"
- board text removed: "@oshpark|@pdp7"
- board text removed: "drew@oshpark.com"
