File: flex-strip-tester.sch (KiCad schematic (older format))
At the start: 5 parts, among them J1 Conn_01x01_Female, J2 Conn_01x01_Female, J3 Conn_01x01_Female

Commit message: try cutout design
Parts:
- J1, J2, J3: footprint touch:TestPoint_Pad_4.0x4.0mm -> Symbol:OSHW-Logo2_7.3x6mm_Copper
Changed lines of the file:
@@
 F 0 "J1" V 3246 2348 50  0000 L CNN
 F 1 "Conn_01x01_Female" V 3337 2348 50  0000 L CNN
-F 2 "touch:TestPoint_Pad_4.0x4.0mm" H 3400 2300 50  0001 C CNN
+F 2 "Symbol:OSHW-Logo2_7.3x6mm_Copper" H 3400 2300 50  0001 C CNN
 F 3 "~" H 3400 2300 50  0001 C CNN
 	1    3400 2300
@@
 F 0 "J2" V 3338 2512 50  0000 R CNN
 F 1 "Conn_01x01_Female" V 3247 2512 50  0000 R CNN
-F 2 "touch:TestPoint_Pad_4.0x4.0mm" H 3400 2600 50  0001 C CNN
+F 2 "Symbol:OSHW-Logo2_7.3x6mm_Copper" H 3400 2600 50  0001 C CNN
 F 3 "~" H 3400 2600 50  0001 C CNN
 	1    3400 2600
@@
 F 0 "J3" V 3138 2712 50  0000 R CNN
 F 1 "Conn_01x01_Female" V 3047 2712 50  0000 R CNN
-F 2 "touch:TestPoint_Pad_4.0x4.0mm" H 3200 2800 50  0001 C CNN
+F 2 "Symbol:OSHW-Logo2_7.3x6mm_Copper" H 3200 2800 50  0001 C CNN
 F 3 "~" H 3200 2800 50  0001 C CNN
 	1    3200 2800
