File: flex-strip-tester-v9b.kicad_pcb (KiCad board)
At the start: 2 copper layers, 67.2 x 11.1 mm, 9 parts, among them J1 Conn_01x01_Female, J2 Conn_01x01_Female

Commit message: refactor the v9 design
Parts:
- removed J1 (x4): Conn_01x01_Female, Symbol:OSHW-Logo2_7.3x6mm_Copper
- removed the J2 at (180.3, 96.9)
- removed the J2 at (180.2, 96.9) (x2)
- added J2 (x2): Conn_01x01_Female, afterdark:OSHW-Logo2_14.6x12mm_Copper, F.Cu at (179.6, 96.5)
- added J2 (x2): Conn_01x01_Female, afterdark:OSHW-Logo2_14.6x12mm_Copper, B.Cu at (179.6, 96.5)
- added J2 (x2): Conn_01x01_Female, afterdark:OSHW-Logo2_14.6x12mm_Copper, F.Cu at (125.2, 96.5)
- added J2 (x2): Conn_01x01_Female, afterdark:OSHW-Logo2_14.6x12mm_Copper, B.Cu at (125.2, 96.5)
- D1: moved to B.Cu
- moved D1 0.80 mm to (153.2, 95.5)
- moved D1 0.70 mm to (153.2, 95.5), turned to 90 degrees
Routing:
- net +3V3: track 39.2 -> 17.7 mm
- net GND: track 26.6 -> 14.4 mm
