File: flex-strip-tester-v2.kicad_pcb (KiCad board)
At the start: 2 copper layers, 67.2 x 11.1 mm, 6 parts, among them J1 Conn_01x01_Female, J2 Conn_01x01_Female

Commit message: add v10 which is being order from oshpark flex
Other:
- net class Default removed
