File: flex-strip-tester-v10.kicad_pcb (KiCad board)
At the start: 2 copper layers, 68.8 x 11.1 mm, 12 parts, among them J2 Conn_01x01_Female

Commit message: osh park freebie version to fab
Parts:
- added REF**: R_0603, Resistor_SMD:R_0603_1608Metric, F.Cu at (132.7, 95.5)
- added REF**: R_0603, Resistor_SMD:R_0603_1608Metric, B.Cu at (174.2, 95.5)
Routing:
- net +3V3: track 34.7 -> 30.2 mm, vias 2 -> 1
- net GND: track 34.6 -> 36.1 mm, vias 2 -> 3
Other:
- board text added: "OSH"
- board text added: "Park"
- board text added: "oshpark.com/flex"
- board text removed: "Drew Fustini"
- board text removed: "drew@ oshpark.com"
