File: flex-strip-tester-v12.kicad_pcb (KiCad board)
At the start: 2 copper layers, 68.8 x 11.1 mm, 15 parts, among them J2 Conn_01x01_Female

Commit message: osh park freebie version to fab
Parts:
- removed Ref**: Val**, flextester:oshpark-v2-park
- removed Ref**: Val**, flextester:oshpark-v2-osh
- moved J2 3.15 mm to (184.4, 96.5) (x4)
- moved J2 2.98 mm to (122.2, 96.5) (x4)
Connections:
- REF** pad 2: GND -> +3V3
Routing:
- net +3V3: track 30.2 -> 36.0 mm, vias 1 -> 2
- net GND: track 37.6 -> 37.4 mm, vias 3 -> 2
Other:
- board size 68.8 x 11.1 mm -> 74.4 x 11.1 mm
- board text added: "OSH"
- board text added: "Park"
- board text removed: "+"
